File: media-keyboard.sch (KiCad schematic (older format))
At the start: 36 parts, among them J1 USB_mini_micro_B, K1 KEYSW, K10 KEYSW, K2 KEYSW, K3 KEYSW, K4 KEYSW, K5 KEYSW, K6 KEYSW, K7 KEYSW, K8 KEYSW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

Commit message: Schematic done!
Parts:
- removed C8: 1u, Capacitor_SMD:C_0805_2012Metric_Pad1.15x1.40mm_HandSolder, symbol Device:C_Small
- removed J1: USB_mini_micro_B, keyboard_parts:USB_miniB_hirose_5S8, symbol keyboard_parts:USB_mini_micro_B
- removed R1, R2: 10k, Resistor_SMD:R_0805_2012Metric_Pad1.15x1.40mm_HandSolder, symbol Device:R
- removed R3, R4: 22, Resistor_SMD:R_0805_2012Metric_Pad1.15x1.40mm_HandSolder, symbol Device:R
- removed SW1: SW_PUSH, Button_Switch_SMD:SW_SPST_TL3342, symbol keyboard_parts:SW_PUSH
- removed X1: 16mhz, Crystal:Crystal_SMD_SeikoEpson_FA238-4Pin_3.2x2.5mm_HandSoldering, symbol Device:Crystal_GND24_Small
- added F1: 500mA, MX_Alps_Hybrid:MX-1U-NoLED, symbol Device:Polyfuse_Small
- added R1, R2: 22, Resistor_SMD:R_0805_2012Metric_Pad1.15x1.40mm_HandSolder, symbol Device:R_Small
- added R3, R4: 10k, Resistor_SMD:R_0805_2012Metric_Pad1.15x1.40mm_HandSolder, symbol Device:R_Small
- added SW1: SW_Push, random-keyboard-parts:SKQG-1155865, symbol Switch:SW_Push
- added USB1: Molex-0548190589, random-keyboard-parts:Molex-0548190589, symbol random-keyboard-parts:Molex-0548190589
- added Y1: 16Mhz, Crystal:Crystal_SMD_3225-4Pin_3.2x2.5mm, symbol Device:Crystal_GND24_Small
- C1, C2: value 22pF -> 0.1uF
- C3, C4: value 0.1uF -> 22uF
- C6: value 0.1uF -> 1uF
- C7: value 4.7uF -> 10uF
- D1, D10, D2, D3, D4, D5, D6, D7, D8, D9: footprint keyboard_parts:D_SOD123_axial -> Diode_SMD:D_SOD-123
- K1, K10, K2, K3, K4, K5, K6, K7, K8, K9: footprint keebs:Mx_Alps_100 -> MX_Alps_Hybrid:MX-1U-NoLED; symbol keyboard_parts:KEYSW -> MX_Alps_Hybrid:MX-NoLED
- U1: symbol keyboard_parts:ATMEGA32U4 -> MCU_Microchip_ATmega:ATmega32U4-AU
Connections:
- net labels added: +5V, D+, D-
- wire segments 95 -> 75
- no-connect marks 19 -> 0
Other:
- moved on the sheet: D1, D10, D2, D3, D4, D5, D6, D7, D8, D9

Commit message: It should work!
Parts:
- added H1, H2, H3, H4: MountingHole, MountingHole:MountingHole_2.2mm_M2, symbol Mechanical:MountingHole
- F1: footprint MX_Alps_Hybrid:MX-1U-NoLED -> Fuse:Fuse_1206_3216Metric
- renumbered C3 to C1, C4 to C2, C6 to C3, C1 to C4, C2 to C5, C5 to C6
Connections:
- net col0: now also U1.31 (PC6)
- net col1: now also U1.30 (PB6)
- net col2: now also U1.29 (PB5)
- net col3: now also U1.28 (PB4)
- net col4: now also U1.27 (PD7)
- net row0: now also U1.25 (PD4)
- net row1: now also U1.26 (PD6)
Changed lines of the file:
@@
 	1500 2300 1200 2300
 $Comp
-L Device:C_Small C6
+L Device:C_Small C3
 U 1 1 5D6C181C
 P 2300 2650
-F 0 "C6" H 2392 2696 50  0000 L CNN
+F 0 "C3" H 2392 2696 50  0000 L CNN
 F 1 "1uF" H 2392 2605 50  0000 L CNN
 F 2 "Capacitor_SMD:C_0805_2012Metric_Pad1.15x1.40mm_HandSolder" H 2300 2650 50  0001 C CNN
@@
 	2300 2500 2650 2500
 $Comp
-L Device:C_Small C2
+L Device:C_Small C5
 U 1 1 5D6C4F32
 P 1300 3750
-F 0 "C2" H 1392 3796 50  0000 L CNN
+F 0 "C5" H 1392 3796 50  0000 L CNN
 F 1 "0.1uF" H 1392 3705 50  0000 L CNN
 F 2 "Capacitor_SMD:C_0805_2012Metric_Pad1.15x1.40mm_HandSolder" H 1300 3750 50  0001 C CNN
@@
 $EndComp
 $Comp
-L Device:C_Small C5
+L Device:C_Small C6
 U 1 1 5D6C5971
 P 1800 3750
-F 0 "C5" H 1892 3796 50  0000 L CNN
+F 0 "C6" H 1892 3796 50  0000 L CNN
 F 1 "0.1uF" H 1892 3705 50  0000 L CNN
 F 2 "Capacitor_SMD:C_0805_2012Metric_Pad1.15x1.40mm_HandSolder" H 1800 3750 50  0001 C CNN
@@
 $EndComp
 $Comp
-L Device:C_Small C1
+L Device:C_Small C4
 U 1 1 5D6C6336
 P 800 3750
-F 0 "C1" H 892 3796 50  0000 L CNN
+F 0 "C4" H 892 3796 50  0000 L CNN
 F 1 "0.1uF" H 892 3705 50  0000 L CNN
 F 2 "Capacitor_SMD:C_0805_2012Metric_Pad1.15x1.40mm_HandSolder" H 800 3750 50  0001 C CNN
@@
 	2650 1400 1950 1400
 $Comp
-L Device:C_Small C3
+L Device:C_Small C1
 U 1 1 5D6DB3AC
 P 1600 1400
-F 0 "C3" V 1550 1250 50  0000 C CNN
+F 0 "C1" V 1550 1250 50  0000 C CNN
 F 1 "22uF" V 1550 1550 50  0000 C CNN
 F 2 "Capacitor_SMD:C_0805_2012Metric_Pad1.15x1.40mm_HandSolder" H 1600 1400 50  0001 C CNN
@@
 $EndComp
 $Comp
-L Device:C_Small C4
+L Device:C_Small C2
 U 1 1 5D6DBD91
 P 1600 1600
-F 0 "C4" V 1550 1450 50  0000 C CNN
+F 0 "C2" V 1550 1450 50  0000 C CNN
 F 1 "22uF" V 1550 1750 50  0000 C CNN
 F 2 "Capacitor_SMD:C_0805_2012Metric_Pad1.15x1.40mm_HandSolder" H 1600 1600 50  0001 C CNN
@@
 F 0 "F1" V 5245 1050 50  0000 C CNN
 F 1 "500mA" V 5336 1050 50  0000 C CNN
-F 2 "MX_Alps_Hybrid:MX-1U-NoLED" H 5500 850 50  0001 L CNN
+F 2 "Fuse:Fuse_1206_3216Metric" H 5500 850 50  0001 L CNN
 F 3 "~" H 5450 1050 50  0001 C CNN
 	1    5450 1050
@@
 	9950 1850 9950 2100
 Connection ~ 9950 2100
+$Comp
+L Mechanical:MountingHole H1
+U 1 1 5D68BBB7
+P 8450 800
+F 0 "H1" H 8550 846 50  0000 L CNN
+F 1 "MountingHole" H 8550 755 50  0000 L CNN
+F 2 "MountingHole:MountingHole_2.2mm_M2" H 8450 800 50  0001 C CNN
+F 3 "~" H 8450 800 50  0001 C CNN
+	1    8450 800
+	1    0    0    -1
+$EndComp
+$Comp
+L Mechanical:MountingHole H2
+U 1 1 5D68BD96
+P 8450 1000
+F 0 "H2" H 8550 1046 50  0000 L CNN
+F 1 "MountingHole" H 8550 955 50  0000 L CNN
+F 2 "MountingHole:MountingHole_2.2mm_M2" H 8450 1000 50  0001 C CNN
+F 3 "~" H 8450 1000 50  0001 C CNN
+	1    8450 1000
+	1    0    0    -1
+$EndComp
+$Comp
+L Mechanical:MountingHole H3
+U 1 1 5D68C0D1
+P 8450 1200
+F 0 "H3" H 8550 1246 50  0000 L CNN
+F 1 "MountingHole" H 8550 1155 50  0000 L CNN
+F 2 "MountingHole:MountingHole_2.2mm_M2" H 8450 1200 50  0001 C CNN
+F 3 "~" H 8450 1200 50  0001 C CNN
+	1    8450 1200
+	1    0    0    -1
+$EndComp
+$Comp
+L Mechanical:MountingHole H4
+U 1 1 5D68C3DE
+P 8450 1400
+F 0 "H4" H 8550 1446 50  0000 L CNN
+F 1 "MountingHole" H 8550 1355 50  0000 L CNN
+F 2 "MountingHole:MountingHole_2.2mm_M2" H 8450 1400 50  0001 C CNN
+F 3 "~" H 8450 1400 50  0001 C CNN
+	1    8450 1400
+	1    0    0    -1
+$EndComp
+Text GLabel 3850 2800 2    50   Input ~ 0
+row0
+Text GLabel 3850 3000 2    50   Input ~ 0
+row1
+Text GLabel 3850 2100 2    50   Input ~ 0
+col0
+Text GLabel 3850 1800 2    50   Input ~ 0
+col1
+Text GLabel 3850 1700 2    50   Input ~ 0
+col2
+Text GLabel 3850 1600 2    50   Input ~ 0
+col3
+Text GLabel 3850 3100 2    50   Input ~ 0
+col4
 $EndSCHEMATC

Commit message: Some routing cleanup
Connections:
- net GND: now also USB1.6 (SHIELD)
- net row0: now also U1.26 (PD6); no longer U1.25 (PD4)
- net row1: now also U1.32 (PC7); no longer U1.26 (PD6)
- no-connect marks 0 -> 20
Changed lines of the file:
@@
 D-
-$Comp
-L random-keyboard-parts:Molex-0548190589 USB1
-U 1 1 5D70026A
-P 4550 1250
-F 0 "USB1" V 5087 1217 60  0000 C CNN
-F 1 "Molex-0548190589" V 4981 1217 60  0000 C CNN
-F 2 "random-keyboard-parts:Molex-0548190589" H 4550 1250 60  0001 C CNN
-F 3 "" H 4550 1250 60  0001 C CNN
-	1    4550 1250
-	0    -1   -1   0
-$EndComp
 $Comp
 L power:VCC #PWR0112
@@
 	1    0    0    -1
 $EndComp
-Text GLabel 3850 2800 2    50   Input ~ 0
+Text GLabel 3850 3000 2    50   Input ~ 0
 row0
-Text GLabel 3850 3000 2    50   Input ~ 0
+Text GLabel 3850 2200 2    50   Input ~ 0
 row1
 Text GLabel 3850 2100 2    50   Input ~ 0
@@
 Text GLabel 3850 3100 2    50   Input ~ 0
 col4
+$Comp
+L power:GND #PWR0115
+U 1 1 5D707628
+P 5000 950
+F 0 "#PWR0115" H 5000 700 50  0001 C CNN
+F 1 "GND" H 5005 777 50  0000 C CNN
+F 2 "" H 5000 950 50  0001 C CNN
+F 3 "" H 5000 950 50  0001 C CNN
+	1    5000 950
+	1    0    0    -1
+$EndComp
+$Comp
+L random-keyboard-parts:Molex-0548190589 USB1
+U 1 1 5D70026A
+P 4550 1250
+F 0 "USB1" V 5087 1217 60  0000 C CNN
+F 1 "Molex-0548190589" V 4981 1217 60  0000 C CNN
+F 2 "random-keyboard-parts:Molex-0548190589" H 4550 1250 60  0001 C CNN
+F 3 "" H 4550 1250 60  0001 C CNN
+	1    4550 1250
+	0    -1   -1   0
+$EndComp
+Wire Wire Line
+	4850 950  5000 950
+NoConn ~ 3850 1200
+NoConn ~ 3850 1300
+NoConn ~ 3850 1400
+NoConn ~ 3850 1500
+NoConn ~ 3850 1900
+NoConn ~ 3850 2400
+NoConn ~ 3850 2500
+NoConn ~ 3850 2600
+NoConn ~ 3850 2700
+NoConn ~ 3850 2900
+NoConn ~ 3850 2800
+NoConn ~ 3850 3400
+NoConn ~ 3850 3600
+NoConn ~ 3850 3700
+NoConn ~ 3850 3800
+NoConn ~ 3850 3900
+NoConn ~ 3850 4000
+NoConn ~ 3850 4100
+NoConn ~ 2650 1800
+NoConn ~ 4850 1350
 $EndSCHEMATC
