File: media-keyboard.kicad_pcb (KiCad board)
At the start: 2 copper layers, 36 parts, among them J1 USB_mini_micro_B, K1 KEYSW, K10 KEYSW, K2 KEYSW, K3 KEYSW, K4 KEYSW, K5 KEYSW, K6 KEYSW, K7 KEYSW, K8 KEYSW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

Commit message: It should work!
Parts:
- removed C8: 1u, Capacitor_SMD:C_0805_2012Metric_Pad1.15x1.40mm_HandSolder
- removed J1: USB_mini_micro_B, keyboard_parts:USB_miniB_hirose_5S8
- removed X1: 16mhz, Crystal:Crystal_SMD_SeikoEpson_FA238-4Pin_3.2x2.5mm_HandSoldering
- added F1: 500mA, Fuse:Fuse_1206_3216Metric, B.Cu at (40.0, 63.8)
- added H1: MountingHole, MountingHole:MountingHole_2.2mm_M2, F.Cu at (40.5, 48.4)
- added H2: MountingHole, MountingHole:MountingHole_2.2mm_M2, F.Cu at (40.5, 80.2)
- added H3: MountingHole, MountingHole:MountingHole_2.2mm_M2, F.Cu at (162.7, 48.4)
- added H4: MountingHole, MountingHole:MountingHole_2.2mm_M2, F.Cu at (162.7, 80.2)
- added USB1: Molex-0548190589, random-keyboard-parts:Molex-0548190589, B.Cu at (58.5, 47.1)
- added Y1: 16Mhz, Crystal:Crystal_SMD_3225-4Pin_3.2x2.5mm, B.Cu at (54.0, 59.5)
- C1, C2: value 22pF -> 22uF
- C3: value 0.1uF -> 1uF
- C7: value 4.7uF -> 10uF
- D1, D10, D2, D3, D4, D5, D6, D7, D8, D9: footprint keyboard_parts:D_SOD123_axial -> Diode_SMD:D_SOD-123
- K1, K10, K2, K3, K4, K5, K6, K7, K8, K9: footprint keebs:Mx_Alps_100 -> MX_Alps_Hybrid:MX-1U-NoLED
- R1, R2: value 10k -> 22
- R3, R4: value 22 -> 10k
- SW1: value SW_PUSH -> SW_Push; footprint Button_Switch_SMD:SW_SPST_TL3342 -> random-keyboard-parts:SKQG-1155865
- moved U1 139.0 mm to (54.0, 72.2)
- moved SW1 133.0 mm to (48.3, 49.5)
- moved R3 117.5 mm to (44.2, 63.3), turned to 270 degrees
- moved R2 113.5 mm to (45.6, 58.8)
- moved R1 110.2 mm to (45.6, 56.5)
- moved C2 107.6 mm to (50.4, 59.4), turned to 270 degrees
- moved C7 103.4 mm to (45.2, 77.6), turned to 270 degrees
- moved C3 99.0 mm to (44.9, 72.1), turned to 180 degrees
- moved C4 95.0 mm to (46.7, 63.3), turned to 90 degrees
- moved C5 89.1 mm to (62.7, 65.3), turned to 90 degrees
- moved C1 87.5 mm to (57.5, 59.4), turned to 90 degrees
- moved R4 85.9 mm to (62.2, 77.6), turned to 90 degrees
- moved C6 84.7 mm to (58.4, 80.5), turned to 180 degrees
- moved D10 65.4 mm to (158.0, 73.8), turned to 90 degrees
- moved D5 63.6 mm to (158.0, 54.8), turned to 90 degrees
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Connections:
- C3 pad 1: GND -> Net-(C3-Pad1)
- C3 pad 2: VCC -> GND
- C4 pad 1: VCC -> +5V
- C5 pad 1: VCC -> +5V
- C6 pad 1: VCC -> +5V
- C7 pad 1: VCC -> +5V
- D1 pad 1: /row0 -> row0
- D10 pad 1: /row1 -> row1
- D2 pad 1: /row0 -> row0
- D3 pad 1: /row0 -> row0
- D4 pad 1: /row0 -> row0
- D5 pad 1: /row0 -> row0
- D6 pad 1: /row1 -> row1
- D7 pad 1: /row1 -> row1
- D8 pad 1: /row1 -> row1
- D9 pad 1: /row1 -> row1
- K1 pad 1: /col0 -> col0
- K10 pad 1: /col4 -> col4
- K2 pad 1: /col1 -> col1
- K3 pad 1: /col2 -> col2
- K4 pad 1: /col3 -> col3
- K5 pad 1: /col4 -> col4
- K6 pad 1: /col0 -> col0
- K7 pad 1: /col1 -> col1
- K8 pad 1: /col2 -> col2
- K9 pad 1: /col3 -> col3
- R1 pad 2: VCC -> D-
- R2 pad 1: GND -> Net-(R2-Pad1)
- R2 pad 2: Net-(R2-Pad2) -> D+
- R3 pad 1: Net-(R3-Pad1) -> +5V
- R3 pad 2: Net-(J1-Pad2) -> Net-(R3-Pad2)
- R4 pad 1: Net-(J1-Pad3) -> GND
- SW1 pad 2: Net-(R1-Pad1) -> Net-(R3-Pad2)
- U1 pad 13: Net-(R1-Pad1) -> Net-(R3-Pad2)
- U1 pad 14: VCC -> +5V
- U1 pad 16: Net-(C1-Pad1) -> Net-(C2-Pad1)
- U1 pad 17: Net-(C2-Pad1) -> Net-(C1-Pad1)
- U1 pad 2: VCC -> +5V
- U1 pad 24: VCC -> +5V
- U1 pad 25: Net-(U1-Pad25) -> row0
- U1 pad 27: Net-(U1-Pad27) -> col4
- U1 pad 28: Net-(U1-Pad28) -> col3
- U1 pad 29: Net-(U1-Pad29) -> col2
- U1 pad 3: Net-(R3-Pad1) -> Net-(R1-Pad1)
- U1 pad 30: Net-(U1-Pad30) -> col1
- U1 pad 31: Net-(U1-Pad31) -> col0
- U1 pad 32: /col4 -> row1
- U1 pad 33: Net-(R2-Pad2) -> Net-(R4-Pad2)
- U1 pad 34: VCC -> +5V
- U1 pad 36: /col3 -> Net-(U1-Pad36)
- U1 pad 37: /col2 -> Net-(U1-Pad37)
- U1 pad 38: /col1 -> Net-(U1-Pad38)
- U1 pad 39: /col0 -> Net-(U1-Pad39)
- U1 pad 4: Net-(R4-Pad2) -> Net-(R2-Pad1)
- U1 pad 40: /row1 -> Net-(U1-Pad40)
- U1 pad 41: /row0 -> Net-(U1-Pad41)
- U1 pad 44: VCC -> +5V
- U1 pad 6: Net-(C8-Pad1) -> Net-(C3-Pad1)
- U1 pad 7: VCC -> +5V
Routing:
- net col4: track 0.00 -> 114.8 mm
- net row0: track 0.00 -> 106.2 mm
- net row1: track 0.00 -> 101.2 mm
- net col3: track 0.00 -> 95.7 mm
- net GND: track 0.00 -> 92.9 mm
- net +5V: track 0.00 -> 85.5 mm, vias 0 -> 7
- net col2: track 0.00 -> 76.6 mm
- net col1: track 0.00 -> 57.5 mm
- net col0: track 0.00 -> 33.1 mm
- net VCC: track 0.00 -> 25.3 mm
- net Net-(R1-Pad1): track 0.00 -> 24.9 mm
- net Net-(R3-Pad2): track 0.00 -> 24.4 mm, vias 0 -> 2
- net Net-(R2-Pad1): track 0.00 -> 22.6 mm
- net D+: track 0.00 -> 15.7 mm
- net D-: track 0.00 -> 14.0 mm
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Other:
- board outline added: 128.6 x 38.9 mm
- net class Default: trace_width 0.25 -> 0.254
- net class Power added: clearance 0.2, trace_width 0.381, via_dia 0.8, via_drill 0.4

Commit message: Some routing cleanup
Parts:
- moved R1 4.49 mm to (50.0, 55.9)
- moved R2 4.49 mm to (50.0, 58.1)
- moved C2 4.13 mm to (53.2, 62.5), turned to 90 degrees
- moved Y1 3.97 mm to (56.5, 62.6)
- moved C1 3.74 mm to (59.7, 62.5)
- moved C4 2.61 mm to (49.2, 62.7), turned to 0 degrees
- moved R3 1.84 mm to (46.0, 63.3)
- moved C5 1.77 mm to (61.9, 66.9)
- moved C6 0.42 mm to (58.2, 80.2)
Connections:
- U1 pad 25: row0 -> Net-(U1-Pad25)
- U1 pad 26: Net-(U1-Pad26) -> row0
- USB1 pad 6: Net-(USB1-Pad6) -> GND
Routing:
- net GND: track 92.9 -> 44.4 mm, vias 0 -> 15
- net Net-(C2-Pad1): track 12.1 -> 6.11 mm
- net D-: track 14.0 -> 9.26 mm
- net D+: track 15.7 -> 11.0 mm
- net Net-(R3-Pad2): track 24.4 -> 20.6 mm
- net Net-(R2-Pad1): track 22.6 -> 25.3 mm
- net Net-(R1-Pad1): track 24.9 -> 27.3 mm
- net col0: track 33.1 -> 31.5 mm
- net Net-(C1-Pad1): track 9.09 -> 8.22 mm
- net +5V: track 85.5 -> 86.0 mm, vias 7 -> 5
- added copper zone on F.Cu, net GND
Other:
- board text added: "RFL switch-a-roo v0.1"
- board text added: "github.com/flexd"

Commit message: Even more cleanup
Parts:
- moved USB1 0.51 mm to (58.5, 47.6)
Routing:
- net GND: track 44.4 -> 34.6 mm
- net VCC: track 25.3 -> 22.9 mm
- net col0: track 31.5 -> 32.0 mm
Changed lines of the file:
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@@
     (thickness 1.6)
     (drawings 10)
-    (tracks 273)
+    (tracks 276)
     (zones 0)
     (modules 40)
@@
       (outputformat 1)
       (mirror false)
-      (drillshape 1)
+      (drillshape 0)
       (scaleselection 1)
-      (outputdirectory ""))
+      (outputdirectory "Gerbers"))
   )
   (net 0 "")
@@
   )
   (module random-keyboard-parts:Molex-0548190589 (layer B.Cu)
-    (at 58.45175 47.0535 270)
+    (at 58.45175 47.5615 270)
     (attr smd)
     (fp_text reference USB1 (at 2.032 0) (layer B.SilkS)
@@
       (effects (font (size 1 1) (thickness 0.15)) (justify mirror))
     )
-    (fp_text value 10uF (at 0 -1.65 90) (layer B.Fab)
+    (fp_text value 10uF (at 2.96175 0.28575 180) (layer B.Fab)
       (effects (font (size 1 1) (thickness 0.15)) (justify mirror))
     )
@@
   (segment (start 43.924 72.136) (end 43.924 70.9115) (width 0.381) (layer B.Cu) (net 1))
   (segment (start 57.89425 61.45) (end 57.615 61.72925) (width 0.381) (layer B.Cu) (net 1))
-  (segment (start 60.05175 51.5535) (end 60.05175 53.4545) (width 0.381) (layer B.Cu) (net 1))
   (segment (start 62.23 78.631) (end 62.23 79.306) (width 0.381) (layer B.Cu) (net 1))
   (segment (start 44.547372 72.759372) (end 43.924 72.136) (width 0.381) (layer B.Cu) (net 1))
@@
   (via (at 61.9125 64.29375) (size 0.8) (drill 0.4) (layers F.Cu B.Cu) (net 1))
   (segment (start 61.9125 65.88125) (end 61.9125 64.29375) (width 0.381) (layer B.Cu) (net 1))
-  (via (at 60.05175 53.4545) (size 0.8) (drill 0.4) (layers F.Cu B.Cu) (net 1))
-  (segment (start 53.12625 47.68) (end 53.18125 47.625) (width 0.381) (layer B.Cu) (net 1))
-  (via (at 53.18125 47.625) (size 0.8) (drill 0.4) (layers F.Cu B.Cu) (net 1))
-  (segment (start 51.36 47.68) (end 53.12625 47.68) (width 0.381) (layer B.Cu) (net 1))
-  (segment (start 54.23025 47.625) (end 54.80175 47.0535) (width 0.381) (layer B.Cu) (net 1))
-  (segment (start 53.18125 47.625) (end 54.23025 47.625) (width 0.381) (layer B.Cu) (net 1))
-  (segment (start 54.80175 47.0535) (end 54.80175 51.5535) (width 0.381) (layer B.Cu) (net 1))
-  (segment (start 62.10175 47.0535) (end 62.10175 51.5535) (width 0.381) (layer B.Cu) (net 1))
+  (via (at 60.071 53.975) (size 0.8) (drill 0.4) (layers F.Cu B.Cu) (net 1))
+  (segment (start 54.23025 48.133) (end 54.80175 47.5615) (width 0.381) (layer B.Cu) (net 1))
   (via (at 53.213 59.944) (size 0.8) (drill 0.4) (layers F.Cu B.Cu) (net 1))
   (segment (start 53.213 61.45) (end 53.213 59.944) (width 0.381) (layer B.Cu) (net 1))
@@
   (segment (start 63.99 78.631) (end 64.008 78.613) (width 0.381) (layer B.Cu) (net 1))
   (segment (start 62.23 78.631) (end 63.99 78.631) (width 0.381) (layer B.Cu) (net 1))
+  (segment (start 54.73825 47.625) (end 54.80175 47.5615) (width 0.381) (layer B.Cu) (net 1))
+  (via (at 52.07 49.403) (size 0.8) (drill 0.4) (layers F.Cu B.Cu) (net 1))
+  (segment (start 51.36 48.693) (end 52.07 49.403) (width 0.381) (layer B.Cu) (net 1))
+  (segment (start 51.36 47.68) (end 51.36 48.693) (width 0.381) (layer B.Cu) (net 1))
+  (segment (start 60.05175 53.95575) (end 60.071 53.975) (width 0.381) (layer B.Cu) (net 1))
+  (segment (start 60.05175 52.0615) (end 60.05175 53.95575) (width 0.381) (layer B.Cu) (net 1))
   (segment (start 59.61925 63.42925) (end 59.69 63.5) (width 0.254) (layer B.Cu) (net 2))
   (segment (start 57.615 63.42925) (end 59.61925 63.42925) (width 0.254) (layer B.Cu) (net 2))
@@
   (segment (start 53.175 63.538) (end 53.213 63.5) (width 0.254) (layer B.Cu) (net 3))
   (segment (start 53.175 66.53125) (end 53.175 63.538) (width 0.254) (layer B.Cu) (net 3))
-  (segment (start 56.85175 52.4285) (end 56.85175 51.5535) (width 0.381) (layer B.Cu) (net 4))
-  (segment (start 56.85175 53.0595) (end 56.44425 53.467) (width 0.381) (layer B.Cu) (net 4))
-  (segment (start 56.85175 51.5535) (end 56.85175 53.0595) (width 0.381) (layer B.Cu) (net 4))
-  (segment (start 40.005 61.626) (end 40.005 62.351) (width 0.381) (layer B.Cu) (net 4))
-  (segment (start 40.005 58.58918) (end 40.005 61.626) (width 0.381) (layer B.Cu) (net 4))
-  (segment (start 45.12718 53.467) (end 40.005 58.58918) (width 0.381) (layer B.Cu) (net 4))
-  (segment (start 56.44425 53.467) (end 45.12718 53.467) (width 0.381) (layer B.Cu) (net 4))
+  (segment (start 56.85175 52.9365) (end 56.85175 52.0615) (width 0.381) (layer B.Cu) (net 4))
+  (segment (start 56.85175 53.5675) (end 56.19025 54.229) (width 0.381) (layer B.Cu) (net 4))
+  (segment (start 56.85175 52.0615) (end 56.85175 53.5675) (width 0.381) (layer B.Cu) (net 4))
+  (segment (start 48.127 54.229) (end 40.005 62.351) (width 0.381) (layer B.Cu) (net 4))
+  (segment (start 56.19025 54.229) (end 48.127 54.229) (width 0.381) (layer B.Cu) (net 4))
   (segment (start 76.31875 50.26875) (end 80.43125 50.26875) (width 0.254) (layer B.Cu) (net 5))
   (segment (start 81.75625 51.59375) (end 81.75625 53.11875) (width 0.254) (layer B.Cu) (net 5))
@@
   (segment (start 69.85 71.4375) (end 70.00875 71.27875) (width 0.254) (layer F.Cu) (net 21))
   (segment (start 69.499788 71.27875) (end 70.00875 71.27875) (width 0.254) (layer B.Cu) (net 21))
-  (segment (start 66.147288 74.63125) (end 69.499788 71.27875) (width 0.254) (layer B.Cu) (net 21))
-  (segment (start 59.675 74.63125) (end 66.147288 74.63125) (width 0.254) (layer B.Cu) (net 21))
+  (segment (start 60.679 74.63125) (end 59.675 74.63125) (width 0.254) (layer B.Cu) (net 21))
+  (segment (start 65.094566 71.27875) (end 61.742066 74.63125) (width 0.254) (layer B.Cu) (net 21))
+  (segment (start 61.742066 74.63125) (end 60.679 74.63125) (width 0.254) (layer B.Cu) (net 21))
+  (segment (start 70.00875 71.27875) (end 65.094566 71.27875) (width 0.254) (layer B.Cu) (net 21))
   (segment (start 83.25625 62.70625) (end 90.36875 69.81875) (width 0.254) (layer B.Cu) (net 22))
   (segment (start 59.675 73.83125) (end 61.9 73.83125) (width 0.254) (layer B.Cu) (net 22))
@@
   (segment (start 120.410817 61.11875) (end 138.81875 61.11875) (width 0.254) (layer B.Cu) (net 25))
   (segment (start 146.20875 52.22875) (end 146.20875 71.27875) (width 0.254) (layer F.Cu) (net 25))
-  (segment (start 57.65175 51.5535) (end 57.65175 52.991368) (width 0.254) (layer B.Cu) (net 26))
   (segment (start 54.763118 55.88) (end 51.027 55.88) (width 0.254) (layer B.Cu) (net 26))
-  (segment (start 57.65175 52.991368) (end 54.763118 55.88) (width 0.254) (layer B.Cu) (net 26))
-  (segment (start 58.45175 52.9325) (end 58.45175 51.5535) (width 0.254) (layer B.Cu) (net 27))
+  (segment (start 55.271118 55.88) (end 54.763118 55.88) (width 0.254) (layer B.Cu) (net 26))
+  (segment (start 57.65175 53.4405) (end 57.658 53.44675) (width 0.254) (layer B.Cu) (net 26))
+  (segment (start 57.65175 52.0615) (end 57.65175 53.4405) (width 0.254) (layer B.Cu) (net 26))
+  (segment (start 57.658 53.493118) (end 55.271118 55.88) (width 0.254) (layer B.Cu) (net 26))
+  (segment (start 57.658 53.44675) (end 57.658 53.493118) (width 0.254) (layer B.Cu) (net 26))
   (segment (start 53.25 58.13425) (end 51.032 58.13425) (width 0.254) (layer B.Cu) (net 27))
-  (segment (start 58.45175 52.9325) (end 53.25 58.13425) (width 0.254) (layer B.Cu) (net 27))
+  (segment (start 53.758 58.13425) (end 53.25 58.13425) (width 0.254) (layer B.Cu) (net 27))
+  (segment (start 58.45175 53.4405) (end 53.758 58.13425) (width 0.254) (layer B.Cu) (net 27))
+  (segment (start 58.45175 52.0615) (end 58.45175 53.4405) (width 0.254) (layer B.Cu) (net 27))
   (segment (start 47.271 73.83125) (end 48.275 73.83125) (width 0.254) (layer B.Cu) (net 28))
   (segment (start 48.275 73.83125) (end 43.35125 73.83125) (width 0.254) (layer B.Cu) (net 28))
